Commit message: Added bringup package and more config/launch files

File: src/yardguard_description/urdf/xacro/yardguard.xacro (robot description, xacro)
@@ -1,109 +1,109 @@
-<?xml version="1.0"?>
-<robot name="yardguard" xmlns:xacro="http://www.ros.org/wiki/xacro">
-    <xacro:property name="base_length" value="0.288" />
-    <xacro:property name="base_width" value="0.240" />
-    <xacro:property name="base_height" value="0.100" />
-    <xacro:property name="wheel_radius" value="0.070" />
-    <xacro:property name="wheel_height" value="0.055" />
-    <xacro:property name="joint_length" value="0.130" />
-    <xacro:property name="joint_width" value="0.155" />
-    <xacro:property name="joint_height" value="0.045" />
-    <material name="grey">
-        <color rgba="0.5 0.5 0.5 1" />
-    </material>
-    <material name="blue">
-        <color rgba="0 0 0.5 1" />
-    </material>
-    <!-- base_footprint (projection of base_link on the ground) -->
-    <link name="base_footprint"/>
-    <joint name="base_joint" type="fixed">
-        <parent link="base_footprint"/>
-        <child link="base_link"/>
-        <origin xyz="0 0 ${((base_height / 2) - .02) + wheel_radius}" rpy="0 0 0"/>
-    </joint>
-    <!-- base_link and base_scan (required for Nav2) -->
-    <link name="base_link">
-        <visual>
-            <geometry>
-                <box size="${base_length} ${base_width} ${base_height}" />
-            </geometry>
-            <origin xyz="0 0 0" rpy="0 0 0" />
-            <material name="blue" />
-        </visual>
-    </link>
-    <joint name="base_scan_joint" type="fixed">
-        <parent link="base_link"/>
-        <child link="base_scan"/>
-        <origin xyz="-${base_length * 0.15} 0 0.075" rpy="0 0 0"/>
-    </joint>
-    <link name="base_scan">
-        <visual>
-            <geometry>
-                <cylinder radius="${wheel_radius / 2}" length="${wheel_height / 2}"/>
-            </geometry>
-            <origin xyz="0 0 0" rpy="0 0 0" />
-            <material name="grey" />
-        </visual>
-    </link>
-    <!-- Wheels (2 differential wheels + 1 caster wheel to keep the balance) -->
-    <joint name="back_left_wheel_joint" type="continuous">
-        <parent link="base_link"/>
-        <child link="back_left_wheel"/>
-        <origin xyz="-${joint_length} ${joint_width} -${joint_height}" rpy="0 0 0"/>
-        <axis xyz="0 1 0"/>
-    </joint>
-    <link name="back_left_wheel">
-        <visual>
-            <geometry>
-                <cylinder radius="${wheel_radius}" length="${wheel_height}"/>
-            </geometry>
-            <origin xyz="0 0 0" rpy="1.57 0 0" />
-            <material name="grey" />
-        </visual>
-    </link>
-    <joint name="back_right_wheel_joint" type="continuous">
-        <parent link="base_link"/>
-        <child link="back_right_wheel"/>
-        <origin xyz="-${joint_length} -${joint_width} -${joint_height}" rpy="0 0 0"/>
-        <axis xyz="0 1 0"/>
-    </joint>
-    <link name="back_right_wheel">
-        <visual>
-            <geometry>
-                <cylinder radius="${wheel_radius}" length="${wheel_height}"/>
-            </geometry>
-            <origin xyz="0 0 0" rpy="1.57 0 0" />
-            <material name="grey" />
-        </visual>
-    </link>
-    <joint name="front_right_wheel_joint" type="continuous">
-        <parent link="base_link"/>
-        <child link="front_right_wheel"/>
-        <origin xyz="${joint_length} -${joint_width} -${joint_height}" rpy="0 0 0"/>
-        <axis xyz="0 1 0"/>
-    </joint>
-    <link name="front_right_wheel">
-        <visual>
-            <geometry>
-                <cylinder radius="${wheel_radius}" length="${wheel_height}"/>
-            </geometry>
-            <origin xyz="0 0 0" rpy="1.57 0 0" />
-            <material name="grey" />
-        </visual>
-    </link>
-    <joint name="front_left_wheel_joint" type="continuous">
-        <parent link="base_link"/>
-        <child link="front_left_wheel"/>
-        <origin xyz="${joint_length} ${joint_width} -${joint_height}" rpy="0 0 0"/>
-        <axis xyz="0 1 0"/>
-    </joint>
-    <link name="front_left_wheel">
-        <visual>
-            <geometry>
-                <cylinder radius="${wheel_radius}" length="${wheel_height}"/>
-            </geometry>
-            <origin xyz="0 0 0" rpy="1.57 0 0" />
-            <material name="grey" />
-        </visual>
-    </link>
+<?xml version="1.0" ?>
+<!-- =================================================================================== -->
+<!-- |    This document was autogenerated by xacro from /home/daniel/projects/yard_guard/src/yardguard_description/urdf/yardguard.urdf | -->
+<!-- |    EDITING THIS FILE BY HAND IS NOT RECOMMENDED                                 | -->
+<!-- =================================================================================== -->
+<!-- =================================================================================== -->
+<!-- |    This document was autogenerated by xacro from /home/daniel/projects/yard_guard/src/yardguard_description/urdf/xacro/yardguard.xacro | -->
+<!-- |    EDITING THIS FILE BY HAND IS NOT RECOMMENDED                                 | -->
+<!-- =================================================================================== -->
+<robot name="yardguard">
+  <material name="grey">
+    <color rgba="0.5 0.5 0.5 1"/>
+  </material>
+  <material name="blue">
+    <color rgba="0 0 0.5 1"/>
+  </material>
+  <!-- base_footprint (projection of base_link on the ground) -->
+  <link name="base_footprint"/>
+  <joint name="base_joint" type="fixed">
+    <parent link="base_footprint"/>
+    <child link="base_link"/>
+    <origin rpy="0 0 0" xyz="0 0 0.1"/>
+  </joint>
+  <!-- base_link and base_scan (required for Nav2) -->
+  <link name="base_link">
+    <visual>
+      <geometry>
+        <box size="0.288 0.24 0.1"/>
+      </geometry>
+      <origin rpy="0 0 0" xyz="0 0 0"/>
+      <material name="blue"/>
+    </visual>
+  </link>
+  <joint name="base_scan_joint" type="fixed">
+    <parent link="base_link"/>
+    <child link="base_scan"/>
+    <origin rpy="0 0 0" xyz="-0.043199999999999995 0 0.075"/>
+  </joint>
+  <link name="base_scan">
+    <visual>
+      <geometry>
+        <cylinder length="0.0275" radius="0.035"/>
+      </geometry>
+      <origin rpy="0 0 0" xyz="0 0 0"/>
+      <material name="grey"/>
+    </visual>
+  </link>
+  <!-- Wheels (2 differential wheels + 1 caster wheel to keep the balance) -->
+  <joint name="back_left_wheel_joint" type="continuous">
+    <parent link="base_link"/>
+    <child link="back_left_wheel"/>
+    <origin rpy="0 0 0" xyz="-0.13 0.155 -0.045"/>
+    <axis xyz="0 1 0"/>
+  </joint>
+  <link name="back_left_wheel">
+    <visual>
+      <geometry>
+        <cylinder length="0.055" radius="0.07"/>
+      </geometry>
+      <origin rpy="1.57 0 0" xyz="0 0 0"/>
+      <material name="grey"/>
+    </visual>
+  </link>
+  <joint name="back_right_wheel_joint" type="continuous">
+    <parent link="base_link"/>
+    <child link="back_right_wheel"/>
+    <origin rpy="0 0 0" xyz="-0.13 -0.155 -0.045"/>
+    <axis xyz="0 1 0"/>
+  </joint>
+  <link name="back_right_wheel">
+    <visual>
+      <geometry>
+        <cylinder length="0.055" radius="0.07"/>
+      </geometry>
+      <origin rpy="1.57 0 0" xyz="0 0 0"/>
+      <material name="grey"/>
+    </visual>
+  </link>
+  <joint name="front_right_wheel_joint" type="continuous">
+    <parent link="base_link"/>
+    <child link="front_right_wheel"/>
+    <origin rpy="0 0 0" xyz="0.13 -0.155 -0.045"/>
+    <axis xyz="0 1 0"/>
+  </joint>
+  <link name="front_right_wheel">
+    <visual>
+      <geometry>
+        <cylinder length="0.055" radius="0.07"/>
+      </geometry>
+      <origin rpy="1.57 0 0" xyz="0 0 0"/>
+      <material name="grey"/>
+    </visual>
+  </link>
+  <joint name="front_left_wheel_joint" type="continuous">
+    <parent link="base_link"/>
+    <child link="front_left_wheel"/>
+    <origin rpy="0 0 0" xyz="0.13 0.155 -0.045"/>
+    <axis xyz="0 1 0"/>
+  </joint>
+  <link name="front_left_wheel">
+    <visual>
+      <geometry>
+        <cylinder length="0.055" radius="0.07"/>
+      </geometry>
+      <origin rpy="1.57 0 0" xyz="0 0 0"/>
+      <material name="grey"/>
+    </visual>
+  </link>
 </robot>
