Commit message: Got the laser scanning working

File: src/yardguard_description/urdf/lidar.xacro (robot description, xacro)
@@ -1,8 +1,6 @@
 <?xml version="1.0" ?>
 <robot xmlns:xacro="www.ros.org">
-  <!-- Define the parent link for the lidar (e.g., base_link or chassis_link) -->
-  <xacro:property name="parent_link_name" value="base_link" />
   <!-- Lidar Link Definition -->
-  <link name="lidar_link">
+  <link name="base_scan">
       <visual>
           <geometry>
@@ -29,30 +27,30 @@
   <!-- Lidar Joint Definition -->
   <joint name="lidar_joint" type="fixed">
-      <parent link="${parent_link_name}"/>
-      <child link="lidar_link"/>
+      <parent link="base_link"/>
+      <child link="base_scan"/>
       <!-- Position the lidar on top of the parent link (adjust xyz values as needed) -->
-      <origin xyz="0.1 0 0.2" rpy="0 0 0"/>
+      <origin xyz="0.08 0 0.1" rpy="0 0 0"/>
   </joint>
-  <gazebo reference="lidar_link">
+  <gazebo reference="base_scan">
       <sensor name="lidar" type="gpu_lidar">
           <always_on>true</always_on>
           <visualize>true</visualize>
-          <pose>-0.064 0 0.121 0 0 0</pose>
-          <update_rate>1</update_rate>
+          <update_rate>10</update_rate>
           <topic>scan</topic>
+          <gz_frame_id>base_scan</gz_frame_id>
           <lidar>
               <scan>
                   <horizontal>
-                      <samples>720</samples>
+                      <samples>360</samples>
                       <resolution>1</resolution>
                       <min_angle>-3.14</min_angle>
                       <max_angle>3.14</max_angle>
                   </horizontal>
-                  <vertical>
+                  <!-- <vertical>
                       <samples>1</samples>
                       <resolution>1</resolution>
                       <min_angle>0.0</min_angle>
                       <max_angle>0.0</max_angle>
-                  </vertical>
+                  </vertical> -->
               </scan>
               <range>

File: src/yardguard_description/urdf/output/yardguard.urdf (robot description, URDF)
Before this commit: robot yardguard, 9 links, 8 joints
Links:
- removed link lidar_link
- added link base_scan, mass 0.1; collision cylinder length=0.04 radius=0.05; visual cylinder length=0.04 radius=0.05
Joints:
- joint lidar_joint: child lidar_link -> base_scan; origin xyz=0.1 0 0.2 rpy=0 0 0 -> xyz=0.08 0 0.1 rpy=0 0 0
