Commit message: fixed build issue

File: src/yardguard_description/urdf/camera.xacro (robot description, xacro)
@@ -1,4 +1,4 @@
 <?xml version="1.0"?>
-<robot xmlns:xacro="http://www.ros.org/wiki/xacro">
+<robot name="yardguard" xmlns:xacro="http://www.ros.org/wiki/xacro">
     <xacro:property name="camera_length" value="0.01" />
     <xacro:property name="camera_width" value="0.05" />

File: src/yardguard_description/urdf/common_properties.xacro (robot description, xacro)
@@ -1,4 +1,9 @@
 <?xml version="1.0"?>
 <robot xmlns:xacro="http://www.ros.org/wiki/xacro">
+  <xacro:property name="base_length" value="0.288" />
+  <xacro:property name="base_width" value="0.24" />
+  <xacro:property name="base_height" value="0.15" />
+    <xacro:property name="wheel_radius" value="0.1" />
+  <xacro:property name="wheel_length" value="0.05" />
     <material name="blue">
         <color rgba="0 0 0.5 1" />

File: src/yardguard_description/urdf/mobile_base.xacro (robot description, xacro)
@@ -1,9 +1,4 @@
 <?xml version="1.0" ?>
 <robot name="yardguard" xmlns:xacro="http://www.ros.org/wiki/xacro">
-  <xacro:property name="base_length" value="0.288" />
-  <xacro:property name="base_width" value="0.24" />
-  <xacro:property name="base_height" value="0.15" />
-  <xacro:property name="wheel_radius" value="0.1" />
-  <xacro:property name="wheel_length" value="0.05" />
   <!-- base_footprint (projection of base_link on the ground) -->
   <link name="base_footprint"/>
