Commit message: intial work

File: src/yardguard_description/urdf/mobile_base.ros2_control.xacro (robot description, xacro)
@@ -11,15 +11,5 @@
             <state_interface name="velocity" />
         </joint>
-        <joint name="front_left_wheel_joint">
-            <command_interface name="velocity" />
-            <state_interface name="position" />
-            <state_interface name="velocity" />
-        </joint>
         <joint name="back_right_wheel_joint">
-            <command_interface name="velocity" />
-            <state_interface name="position" />
-            <state_interface name="velocity" />
-        </joint>
-        <joint name="front_right_wheel_joint">
             <command_interface name="velocity" />
             <state_interface name="position" />

File: src/yardguard_description/urdf/mobile_base_gazebo.xacro (robot description, xacro)
@@ -11,6 +11,4 @@
             <left_joint>back_left_wheel_joint</left_joint>
             <right_joint>back_right_wheel_joint</right_joint>
-            <left_joint>front_left_wheel_joint</left_joint>
-            <right_joint>front_right_wheel_joint</right_joint>
             <wheel_separation>0.45</wheel_separation>
             <wheel_radius>0.1</wheel_radius>
@@ -25,6 +23,4 @@
             <joint_name>back_left_wheel_joint</joint_name>
             <joint_name>back_right_wheel_joint</joint_name>
-            <joint_name>front_left_wheel_joint</joint_name>
-            <joint_name>front_right_wheel_joint</joint_name>
         </plugin>
     </gazebo>

File: src/yardguard_description/urdf/output/yardguard.urdf (robot description, URDF)
Before this commit: robot yardguard, 9 links, 8 joints
Joints:
- joint front_left_wheel_joint: type continuous -> fixed
- joint front_right_wheel_joint: type continuous -> fixed
