Commit message: got the ros code working with odrive well, turning works well now

File: src/yardguard_description/urdf/common_properties.xacro (robot description, xacro)
@@ -4,6 +4,6 @@
   <xacro:property name="base_width" value="0.24" />
   <xacro:property name="base_height" value="0.15" />
-    <xacro:property name="wheel_radius" value="0.1" />
-  <xacro:property name="wheel_length" value="0.05" />
+    <xacro:property name="wheel_radius" value="0.065" />
+  <xacro:property name="wheel_length" value="0.1" />
     <material name="blue">
         <color rgba="0 0 0.5 1" />

File: src/yardguard_description/urdf/output/yardguard.urdf (robot description, URDF)
Before this commit: robot yardguard, 9 links, 8 joints
Links:
- link back_left_wheel: geometry collision sphere radius=0.065; visual cylinder length=0.1 radius=0.065
- link back_right_wheel: geometry collision sphere radius=0.065; visual cylinder length=0.1 radius=0.065
- link front_left_wheel: geometry collision sphere radius=0.065; visual cylinder length=0.1 radius=0.065
- link front_right_wheel: geometry collision sphere radius=0.065; visual cylinder length=0.1 radius=0.065
Joints:
- joint base_joint: origin xyz=0 0 0.135 rpy=0 0 0 -> xyz=0 0 0.1 rpy=0 0 0
