Commit message: Split the xacro files into multiple files

File: src/yardguard_description/urdf/mobile_base.xacro (robot description, xacro)
@@ -1,28 +1,9 @@
 <?xml version="1.0" ?>
-<!-- =================================================================================== -->
-<!-- |    This document was autogenerated by xacro from /home/daniel/projects/yard_guard/src/yardguard_description/urdf/yardguard.xacro | -->
-<!-- |    EDITING THIS FILE BY HAND IS NOT RECOMMENDED                                 | -->
-<!-- =================================================================================== -->
-<robot name="yardguard">
-  <!-- <gazebo reference="caster_wheel_link">
-        <mu1 value="0.1" />
-        <mu2 value="0.1" />
-    </gazebo> -->
-  <gazebo>
-    <plugin filename="gz-sim-diff-drive-system" name="gz::sim::systems::DiffDrive">
-      <left_joint>back_left_wheel_joint</left_joint>
-      <right_joint>back_right_wheel_joint</right_joint>
-      <wheel_separation>0.45</wheel_separation>
-      <wheel_radius>0.1</wheel_radius>
-      <frame_id>odom</frame_id>
-      <child_frame_id>base_footprint</child_frame_id>
-    </plugin>
-  </gazebo>
-  <gazebo>
-    <plugin filename="gz-sim-joint-state-publisher-system" name="gz::sim::systems::JointStatePublisher">
-      <joint_name>back_left_wheel_joint</joint_name>
-      <joint_name>back_right_wheel_joint</joint_name>
-    </plugin>
-  </gazebo>
+<robot name="yardguard" xmlns:xacro="http://www.ros.org/wiki/xacro">
+  <xacro:property name="base_length" value="0.288" />
+  <xacro:property name="base_width" value="0.24" />
+  <xacro:property name="base_height" value="0.1" />
+  <xacro:property name="wheel_radius" value="0.1" />
+  <xacro:property name="wheel_length" value="0.05" />
   <!-- base_footprint (projection of base_link on the ground) -->
   <link name="base_footprint"/>
@@ -36,5 +17,5 @@
     <visual>
       <geometry>
-        <box size="0.288 0.24 0.1 "/>
+        <box size="${base_length} ${base_width} ${base_height} "/>
       </geometry>
       <origin rpy="0 0 0" xyz="0 0 0"/>
@@ -66,5 +47,5 @@
     <visual>
       <geometry>
-        <cylinder length="0.05" radius="0.1"/>
+        <cylinder length="${wheel_length}" radius="${wheel_radius}"/>
       </geometry>
       <origin rpy="1.57 0 0" xyz="0 0 0"/>
@@ -81,5 +62,5 @@
     <visual>
       <geometry>
-        <cylinder length="0.05" radius="0.1"/>
+        <cylinder length="${wheel_length}" radius="${wheel_radius}"/>
       </geometry>
       <origin rpy="1.57 0 0" xyz="0 0 0"/>
@@ -96,5 +77,5 @@
     <visual>
       <geometry>
-        <cylinder length="0.05" radius="0.1"/>
+        <cylinder length="${wheel_length}" radius="${wheel_radius}"/>
       </geometry>
       <origin rpy="1.57 0 0" xyz="0 0 0"/>
@@ -111,5 +92,5 @@
     <visual>
       <geometry>
-        <cylinder length="0.05" radius="0.1"/>
+        <cylinder length="${wheel_length}" radius="${wheel_radius}"/>
       </geometry>
       <origin rpy="1.57 0 0" xyz="0 0 0"/>

File: src/yardguard_description/urdf/yardguard.xacro (robot description, xacro)
@@ -3,106 +3,4 @@
   <xacro:include filename="mobile_base_gazebo.xacro" />
   <!-- <xacro:include filename="common_properties.xacro" /> -->
-  <xacro:property name="base_length" value="0.288" />
-  <xacro:property name="base_width" value="0.24" />
-  <xacro:property name="base_height" value="0.1" />
-  <xacro:property name="wheel_radius" value="0.1" />
-  <xacro:property name="wheel_length" value="0.05" />
-  <material name="grey">
-    <color rgba="0.5 0.5 0.5 1"/>
-  </material>
-  <material name="blue">
-    <color rgba="0 0 0.5 1"/>
-  </material>
-  <!-- base_footprint (projection of base_link on the ground) -->
-  <link name="base_footprint"/>
-  <joint name="base_joint" type="fixed">
-    <parent link="base_footprint"/>
-    <child link="base_link"/>
-    <origin rpy="0 0 0" xyz="0 0 0.1"/>
-  </joint>
-  <!-- base_link and base_scan (required for Nav2) -->
-  <link name="base_link">
-    <visual>
-      <geometry>
-        <box size="${base_length} ${base_width} ${base_height} "/>
-      </geometry>
-      <origin rpy="0 0 0" xyz="0 0 0"/>
-      <material name="blue"/>
-    </visual>
-  </link>
-  <joint name="base_scan_joint" type="fixed">
-    <parent link="base_link"/>
-    <child link="base_scan"/>
-    <origin rpy="0 0 0" xyz="-0.043199999999999995 0 0.075"/>
-  </joint>
-  <link name="base_scan">
-    <visual>
-      <geometry>
-        <cylinder length="0.0275" radius="0.035"/>
-      </geometry>
-      <origin rpy="0 0 0" xyz="0 0 0"/>
-      <material name="grey"/>
-    </visual>
-  </link>
-  <!-- Wheels (2 differential wheels + 1 caster wheel to keep the balance) -->
-  <joint name="back_left_wheel_joint" type="continuous">
-    <parent link="base_link"/>
-    <child link="back_left_wheel"/>
-    <origin rpy="0 0 0" xyz="-0.13 0.155 -0.045"/>
-    <axis xyz="0 1 0"/>
-  </joint>
-  <link name="back_left_wheel">
-    <visual>
-      <geometry>
-        <cylinder length="${wheel_length}" radius="${wheel_radius}"/>
-      </geometry>
-      <origin rpy="1.57 0 0" xyz="0 0 0"/>
-      <material name="grey"/>
-    </visual>
-  </link>
-  <joint name="back_right_wheel_joint" type="continuous">
-    <parent link="base_link"/>
-    <child link="back_right_wheel"/>
-    <origin rpy="0 0 0" xyz="-0.13 -0.155 -0.045"/>
-    <axis xyz="0 1 0"/>
-  </joint>
-  <link name="back_right_wheel">
-    <visual>
-      <geometry>
-        <cylinder length="${wheel_length}" radius="${wheel_radius}"/>
-      </geometry>
-      <origin rpy="1.57 0 0" xyz="0 0 0"/>
-      <material name="grey"/>
-    </visual>
-  </link>
-  <joint name="front_right_wheel_joint" type="continuous">
-    <parent link="base_link"/>
-    <child link="front_right_wheel"/>
-    <origin rpy="0 0 0" xyz="0.13 -0.155 -0.045"/>
-    <axis xyz="0 1 0"/>
-  </joint>
-  <link name="front_right_wheel">
-    <visual>
-      <geometry>
-        <cylinder length="${wheel_length}" radius="${wheel_radius}"/>
-      </geometry>
-      <origin rpy="1.57 0 0" xyz="0 0 0"/>
-      <material name="grey"/>
-    </visual>
-  </link>
-  <joint name="front_left_wheel_joint" type="continuous">
-    <parent link="base_link"/>
-    <child link="front_left_wheel"/>
-    <origin rpy="0 0 0" xyz="0.13 0.155 -0.045"/>
-    <axis xyz="0 1 0"/>
-  </joint>
-  <link name="front_left_wheel">
-    <visual>
-      <geometry>
-        <cylinder length="${wheel_length}" radius="${wheel_radius}"/>
-      </geometry>
-      <origin rpy="1.57 0 0" xyz="0 0 0"/>
-      <material name="grey"/>
-    </visual>
-  </link>
+  <xacro:include filename="mobile_base.xacro" />
 </robot>

Commit message: added collision tags and a test dpt world

File: src/yardguard_description/urdf/mobile_base.xacro (robot description, xacro)
@@ -22,4 +22,12 @@
       <material name="blue"/>
     </visual>
+    <collision>
+        <geometry>
+            <box size="${base_length} ${base_width} ${base_height}" />
+        </geometry>
+        <origin xyz="0 0 ${base_height / 2.0}" rpy="0 0 0" />
+    </collision>
+    <xacro:box_inertia m="5.0" x="${base_length}" y="${base_width}" z="${base_height}"
+                           o_xyz="0 0 ${base_height / 2.0}" o_rpy="0 0 0" />
   </link>
   <joint name="base_scan_joint" type="fixed">
@@ -52,4 +60,12 @@
       <material name="grey"/>
     </visual>
+    <collision>
+        <geometry>
+            <sphere radius="${wheel_radius}" />
+        </geometry>
+        <origin xyz="0 0 0" rpy="0 0 0" />
+    </collision>
+    <xacro:cylinder_inertia m="1.0" r="${wheel_radius}" l="${wheel_length}"
+                            o_xyz="0 0 0" o_rpy="${pi / 2.0} 0 0" />
   </link>
   <joint name="back_right_wheel_joint" type="continuous">
@@ -67,4 +83,12 @@
       <material name="grey"/>
     </visual>
+    <collision>
+        <geometry>
+            <sphere radius="${wheel_radius}" />
+        </geometry>
+        <origin xyz="0 0 0" rpy="0 0 0" />
+    </collision>
+    <xacro:cylinder_inertia m="1.0" r="${wheel_radius}" l="${wheel_length}"
+                            o_xyz="0 0 0" o_rpy="${pi / 2.0} 0 0" />
   </link>
   <joint name="front_right_wheel_joint" type="continuous">
@@ -82,4 +106,12 @@
       <material name="grey"/>
     </visual>
+    <collision>
+        <geometry>
+            <sphere radius="${wheel_radius}" />
+        </geometry>
+        <origin xyz="0 0 0" rpy="0 0 0" />
+    </collision>
+    <xacro:cylinder_inertia m="1.0" r="${wheel_radius}" l="${wheel_length}"
+                            o_xyz="0 0 0" o_rpy="${pi / 2.0} 0 0" />
   </link>
   <joint name="front_left_wheel_joint" type="continuous">
@@ -97,4 +129,12 @@
       <material name="grey"/>
     </visual>
+    <collision>
+        <geometry>
+            <sphere radius="${wheel_radius}" />
+        </geometry>
+        <origin xyz="0 0 0" rpy="0 0 0" />
+    </collision>
+    <xacro:cylinder_inertia m="1.0" r="${wheel_radius}" l="${wheel_length}"
+                            o_xyz="0 0 0" o_rpy="${pi / 2.0} 0 0" />
   </link>
 </robot>

File: src/yardguard_description/urdf/output/yardguard.urdf (robot description, URDF)
Before this commit: robot yardguard, 7 links, 6 joints
Links:
- link back_left_wheel: mass None -> 1.0; geometry collision sphere radius=0.1; visual cylinder length=0.05 radius=0.1
- link back_right_wheel: mass None -> 1.0; geometry collision sphere radius=0.1; visual cylinder length=0.05 radius=0.1
- link base_link: mass None -> 5.0; geometry collision box size=0.288 0.24 0.1; visual box size=0.288 0.24 0.1
- link front_left_wheel: mass None -> 1.0; geometry collision sphere radius=0.1; visual cylinder length=0.05 radius=0.1
- link front_right_wheel: mass None -> 1.0; geometry collision sphere radius=0.1; visual cylinder length=0.05 radius=0.1

File: src/yardguard_description/urdf/yardguard.xacro (robot description, xacro)
@@ -2,5 +2,5 @@
 <robot name="yardguard" xmlns:xacro="http://www.ros.org/wiki/xacro">
   <xacro:include filename="mobile_base_gazebo.xacro" />
-  <!-- <xacro:include filename="common_properties.xacro" /> -->
+  <xacro:include filename="common_properties.xacro" />
   <xacro:include filename="mobile_base.xacro" />
 </robot>

Commit message: Got the robot working in gazebo with teleop_keyboard

File: src/yardguard_description/urdf/mobile_base.xacro (robot description, xacro)
@@ -11,5 +11,5 @@
     <parent link="base_footprint"/>
     <child link="base_link"/>
-    <origin rpy="0 0 0" xyz="0 0 ${wheel_radius + 0.037}"/>
+    <origin rpy="0 0 0" xyz="0 0 ${wheel_radius + 0.035}"/>
   </joint>
   <!-- base_link and base_scan (required for Nav2) -->

File: src/yardguard_description/urdf/output/yardguard.urdf (robot description, URDF)
Before this commit: robot yardguard, 7 links, 6 joints
Joints:
- joint base_joint: origin xyz=0 0 0.137 rpy=0 0 0 -> xyz=0 0 0.135 rpy=0 0 0

File: src/yardguard_description/urdf/yardguard.xacro (robot description, xacro)
@@ -1,6 +1,6 @@
 <?xml version="1.0" ?>
 <robot name="yardguard" xmlns:xacro="http://www.ros.org/wiki/xacro">
-  <xacro:include filename="mobile_base_gazebo.xacro" />
   <xacro:include filename="common_properties.xacro" />
   <xacro:include filename="mobile_base.xacro" />
+  <xacro:include filename="mobile_base_gazebo.xacro" />
 </robot>

Commit message: fixed the robot model not connected to tf map/odom

File: src/yardguard_description/urdf/mobile_base.xacro (robot description, xacro)
@@ -41,5 +41,5 @@
   </link> -->
   <!-- Wheels (2 differential wheels + 1 caster wheel to keep the balance) -->
-  <joint name="back_left_wheel_joint" type="continuous">
+  <joint name="back_left_wheel_joint" type="fixed">
     <parent link="base_link"/>
     <child link="back_left_wheel"/>
@@ -64,5 +64,5 @@
                             o_xyz="0 0 0" o_rpy="${pi / 2.0} 0 0" />
   </link>
-  <joint name="back_right_wheel_joint" type="continuous">
+  <joint name="back_right_wheel_joint" type="fixed">
     <parent link="base_link"/>
     <child link="back_right_wheel"/>
@@ -87,5 +87,5 @@
                             o_xyz="0 0 0" o_rpy="${pi / 2.0} 0 0" />
   </link>
-  <joint name="front_right_wheel_joint" type="continuous">
+  <joint name="front_right_wheel_joint" type="fixed">
     <parent link="base_link"/>
     <child link="front_right_wheel"/>
@@ -110,5 +110,5 @@
                             o_xyz="0 0 0" o_rpy="${pi / 2.0} 0 0" />
   </link>
-  <joint name="front_left_wheel_joint" type="continuous">
+  <joint name="front_left_wheel_joint" type="fixed">
     <parent link="base_link"/>
     <child link="front_left_wheel"/>

File: src/yardguard_description/urdf/output/yardguard.urdf (robot description, URDF)
Before this commit: robot yardguard, 9 links, 8 joints
Joints:
- joint back_left_wheel_joint: type continuous -> fixed
- joint back_right_wheel_joint: type continuous -> fixed
- joint front_left_wheel_joint: type continuous -> fixed
- joint front_right_wheel_joint: type continuous -> fixed

Commit message: made progress

File: src/yardguard_description/urdf/mobile_base.xacro (robot description, xacro)
@@ -41,5 +41,5 @@
   </link> -->
   <!-- Wheels (2 differential wheels + 1 caster wheel to keep the balance) -->
-  <joint name="back_left_wheel_joint" type="fixed">
+  <joint name="back_left_wheel_joint" type="continuous">
     <parent link="base_link"/>
     <child link="back_left_wheel"/>
@@ -64,5 +64,5 @@
                             o_xyz="0 0 0" o_rpy="${pi / 2.0} 0 0" />
   </link>
-  <joint name="back_right_wheel_joint" type="fixed">
+  <joint name="back_right_wheel_joint" type="continuous">
     <parent link="base_link"/>
     <child link="back_right_wheel"/>
@@ -87,5 +87,5 @@
                             o_xyz="0 0 0" o_rpy="${pi / 2.0} 0 0" />
   </link>
-  <joint name="front_right_wheel_joint" type="fixed">
+  <joint name="front_right_wheel_joint" type="continuous">
     <parent link="base_link"/>
     <child link="front_right_wheel"/>
@@ -110,5 +110,5 @@
                             o_xyz="0 0 0" o_rpy="${pi / 2.0} 0 0" />
   </link>
-  <joint name="front_left_wheel_joint" type="fixed">
+  <joint name="front_left_wheel_joint" type="continuous">
     <parent link="base_link"/>
     <child link="front_left_wheel"/>

File: src/yardguard_description/urdf/output/yardguard.urdf (robot description, URDF)
Before this commit: robot yardguard, 9 links, 8 joints
Joints:
- joint back_left_wheel_joint: type fixed -> continuous
- joint back_right_wheel_joint: type fixed -> continuous
- joint front_left_wheel_joint: type fixed -> continuous
- joint front_right_wheel_joint: type fixed -> continuous
