Commit message: made some progress on getting lidar scanner hooked up but still not working 100%

File: src/yardguard_description/urdf/output/yardguard.urdf (robot description, URDF)
Before this commit: robot yardguard, 9 links, 8 joints
Links:
- removed link base_scan
- added link lidar_link, mass 0.1; collision cylinder length=0.04 radius=0.05; visual cylinder length=0.04 radius=0.05
Joints:
- removed joint base_scan_joint
- added joint lidar_joint: type fixed, parent base_link, child lidar_link, origin xyz=0.1 0 0.2 rpy=0 0 0

Commit message: Got the odrive code integrated with yardguard

File: src/yardguard_description/urdf/output/yardguard.urdf (robot description, URDF)
Before this commit: robot yardguard, 9 links, 8 joints
Joints:
- joint front_left_wheel_joint: type fixed -> continuous
- joint front_right_wheel_joint: type fixed -> continuous

File: src/yardguard_description/urdf/yardguard.xacro (robot description, xacro)
@@ -1,9 +1,12 @@
 <?xml version="1.0" ?>
 <robot name="yardguard" xmlns:xacro="http://www.ros.org/wiki/xacro">
+  <xacro:arg name="prefix" default="back" />
+  <xacro:arg name="use_mock_hardware" default="false" />
   <xacro:include filename="common_properties.xacro" />
-  <xacro:include filename="mobile_base_gazebo.xacro" />
+  <xacro:include filename="diffbot.ros2_control.xacro" />
   <xacro:include filename="camera.xacro" />
   <xacro:include filename="lidar.xacro" />
-  <xacro:include filename="mobile_base.ros2_control.xacro" />
   <xacro:include filename="mobile_base.xacro" />
+  <xacro:diffbot_ros2_control
+    name="DiffBot" prefix="$(arg prefix)" use_mock_hardware="$(arg use_mock_hardware)"/>
 </robot>
